File: Projects/MyProjects/ESC_Driver/Design/rev01/rev01_1/ESC_Driver/ESC_Driver.kicad_sch (KiCad schematic)
At the start: 0 parts

Commit message: Update 2
Create a project ESC.
Maked a diagram.
Other:
- added sheet BLOCK_DIAGRAM (BLOCK_DIAGRAM.kicad_sch)
- added sheet CAN (CAN.kicad_sch)
- added sheet FILTERS (FILTERS.kicad_sch)
- added sheet MCU (MCU_sch.kicad_sch)
- added sheet MECHANICAL (MECHANICAL.kicad_sch)
- added sheet MOSFET DRIVER (MOSFET_DRIVER.kicad_sch)
- added sheet MOSFETs (MOSFETs.kicad_sch)
- added sheet OVERVIEW (OVERVIEW.kicad_sch)
- note added: "ESC Driver rev01_01"
Changed lines of the file:
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@@
     (comment 3 "Tomasz Piskor")
+  )
+  (text "ESC Driver rev01_01" (at 78.74 27.94 0)
+    (effects (font (size 10 10) (thickness 2) bold) (justify left bottom))
+  )
+  (sheet (at 109.22 68.58) (size 26.67 25.4) (fields_autoplaced)
+    (stroke (width 0.1524) (type solid))
+    (fill (color 0 0 0 0.0000))
+    (property "Sheetname" "MOSFETs" (at 109.22 67.8684 0)
+      (effects (font (size 1.27 1.27)) (justify left bottom))
+    )
+    (property "Sheetfile" "MOSFETs.kicad_sch" (at 109.22 94.5646 0)
+      (effects (font (size 1.27 1.27)) (justify left top))
+    )
+    (instances
+      (project "ESC_Driver"
+        (path "/e63e39d7-6ac0-4ffd-8aa3-1841a4541b55" (page "4"))
+      )
+    )
+  )
+  (sheet (at 71.12 41.91) (size 27.94 21.59) (fields_autoplaced)
+    (stroke (width 0.1524) (type solid))
+    (fill (color 0 0 0 0.0000))
+    (property "Sheetname" "BLOCK_DIAGRAM" (at 71.12 41.1984 0)
+      (effects (font (size 1.27 1.27)) (justify left bottom))
+    )
+    (property "Sheetfile" "BLOCK_DIAGRAM.kicad_sch" (at 71.12 64.0846 0)
+      (effects (font (size 1.27 1.27)) (justify left top))
+    )
+    (instances
+      (project "ESC_Driver"
+        (path "/e63e39d7-6ac0-4ffd-8aa3-1841a4541b55" (page "8"))
+      )
+    )
+  )
+  (sheet (at 33.02 41.91) (size 27.94 21.59) (fields_autoplaced)
+    (stroke (width 0.1524) (type solid))
+    (fill (color 0 0 0 0.0000))
+    (property "Sheetname" "OVERVIEW" (at 33.02 41.1984 0)
+      (effects (font (size 1.27 1.27)) (justify left bottom))
+    )
+    (property "Sheetfile" "OVERVIEW.kicad_sch" (at 33.02 64.0846 0)
+      (effects (font (size 1.27 1.27)) (justify left top))
+    )
+    (instances
+      (project "ESC_Driver"
+        (path "/e63e39d7-6ac0-4ffd-8aa3-1841a4541b55" (page "7"))
+      )
+    )
+  )
+  (sheet (at 33.02 68.58) (size 24.13 24.13) (fields_autoplaced)
+    (stroke (width 0.1524) (type solid))
+    (fill (color 0 0 0 0.0000))
+    (property "Sheetname" "MCU" (at 33.02 67.8684 0)
+      (effects (font (size 1.27 1.27)) (justify left bottom))
+    )
+    (property "Sheetfile" "MCU_sch.kicad_sch" (at 33.02 93.2946 0)
+      (effects (font (size 1.27 1.27)) (justify left top))
+    )
+    (instances
+      (project "ESC_Driver"
+        (path "/e63e39d7-6ac0-4ffd-8aa3-1841a4541b55" (page "2"))
+      )
+    )
+  )
+  (sheet (at 33.02 100.33) (size 24.13 25.4) (fields_autoplaced)
+    (stroke (width 0.1524) (type solid))
+    (fill (color 0 0 0 0.0000))
+    (property "Sheetname" "MECHANICAL" (at 33.02 99.6184 0)
+      (effects (font (size 1.27 1.27)) (justify left bottom))
+    )
+    (property "Sheetfile" "MECHANICAL.kicad_sch" (at 33.02 126.3146 0)
+      (effects (font (size 1.27 1.27)) (justify left top))
+    )
+    (instances
+      (project "ESC_Driver"
+        (path "/e63e39d7-6ac0-4ffd-8aa3-1841a4541b55" (page "9"))
+      )
+    )
+  )
+  (sheet (at 143.51 68.58) (size 25.4 25.4) (fields_autoplaced)
+    (stroke (width 0.1524) (type solid))
+    (fill (color 0 0 0 0.0000))
+    (property "Sheetname" "CAN" (at 143.51 67.8684 0)
+      (effects (font (size 1.27 1.27)) (justify left bottom))
+    )
+    (property "Sheetfile" "CAN.kicad_sch" (at 143.51 94.5646 0)
+      (effects (font (size 1.27 1.27)) (justify left top))
+    )
+    (instances
+      (project "ESC_Driver"
+        (path "/e63e39d7-6ac0-4ffd-8aa3-1841a4541b55" (page "5"))
+      )
+    )
+  )
+  (sheet (at 179.07 68.58) (size 25.4 25.4) (fields_autoplaced)
+    (stroke (width 0.1524) (type solid))
+    (fill (color 0 0 0 0.0000))
+    (property "Sheetname" "FILTERS" (at 179.07 67.8684 0)
+      (effects (font (size 1.27 1.27)) (justify left bottom))
+    )
+    (property "Sheetfile" "FILTERS.kicad_sch" (at 179.07 94.5646 0)
+      (effects (font (size 1.27 1.27)) (justify left top))
+    )
+    (instances
+      (project "ESC_Driver"
+        (path "/e63e39d7-6ac0-4ffd-8aa3-1841a4541b55" (page "6"))
+      )
+    )
+  )
+  (sheet (at 71.12 68.58) (size 24.13 24.13) (fields_autoplaced)
+    (stroke (width 0.1524) (type solid))
+    (fill (color 0 0 0 0.0000))
+    (property "Sheetname" "MOSFET DRIVER" (at 71.12 67.8684 0)
+      (effects (font (size 1.27 1.27)) (justify left bottom))
+    )
+    (property "Sheetfile" "MOSFET_DRIVER.kicad_sch" (at 71.12 93.2946 0)
+      (effects (font (size 1.27 1.27)) (justify left top))
+    )
+    (instances
+      (project "ESC_Driver"
+        (path "/e63e39d7-6ac0-4ffd-8aa3-1841a4541b55" (page "3"))
+      )
+    )
   )
   (sheet_instances
